File: 555_556_Tester 2.sch (EAGLE design)
At the start: 19 parts, among them IC1 556, IC2 555, J2 POWER_JACKPTH

Commit message: Revisions
Parts:
- removed IC2: 555, linear:NE555N
- added 555: 555, SparkFun-AnalogIC:NE555KIT
Connections:
- net 556IC11 renamed CV2
- net 556IC13 renamed DIS2
- net 556IC9 renamed OUT2
- net TRIG2 renamed THR2_TRIG2
- removed net +5V: IC1.RST, IC1.RST2, IC1.VCC, IC2.R, IC2.V+, J2.PWR, R1.2, R4.2, R5.2, R6.2
- removed net 556IC5: D1.C, IC1.OUT, IC2.Q, R2.2
- removed net THR: C1.+, IC1.THR, IC1.TRIG, IC2.THR, IC2.TR, R8.1
- new net OUT: 555.OUT, D1.C, IC1.OUT, R2.2
- new net THR_TRIG: 555.TRE, 555.TRI, C1.+, IC1.THR, IC1.TRIG, R8.1
- new net VCC+: 555.VCC+, IC1.RST, IC1.RST2, IC1.VCC, J2.PWR, R1.2, R4.2, R5.2, R6.2
- net CV: now also 555.CON; no longer IC2.CV
- net DIS: now also 555.DIS; no longer IC2.DIS
- net GND: now also 555./RES, 555.GND; no longer IC2.GND
Changed lines of the file:
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@@
 <layer number="19" name="Unrouted" color="6" fill="1" visible="yes" active="no"/>
 <layer number="20" name="Dimension" color="15" fill="1" visible="yes" active="no"/>
-<layer number="21" name="tPlace" color="7" fill="1" visible="yes" active="no"/>
-<layer number="22" name="bPlace" color="7" fill="1" visible="yes" active="no"/>
+<layer number="21" name="tPlace" color="48" fill="1" visible="yes" active="no"/>
+<layer number="22" name="bPlace" color="42" fill="1" visible="yes" active="no"/>
 <layer number="23" name="tOrigins" color="15" fill="1" visible="yes" active="no"/>
 <layer number="24" name="bOrigins" color="15" fill="1" visible="yes" active="no"/>
@@
 <part name="C4" library="adafruit" deviceset="C-US" device="025-025X050" value="10nF"/>
 <part name="J2" library="SparkFun-Connectors" deviceset="POWER_JACK" device="PTH"/>
-<part name="IC2" library="linear" deviceset="*555" device="N" technology="NE" value="555"/>
+<part name="555" library="SparkFun-AnalogIC" deviceset="NE555" device="KIT" value="555"/>
 </parts>
 <sheets>
@@
 <instance part="C4" gate="G$1" x="82.55" y="-27.94"/>
 <instance part="J2" gate="G$1" x="7.62" y="20.32"/>
-<instance part="IC2" gate="A" x="69.85" y="-6.35"/>
+<instance part="555" gate="G$1" x="69.85" y="-6.35"/>
 </instances>
 <busses>
-<bus name="556IC[1..14],GND,DIS,THR,CV,RST,OUT,TRIG,VCC,DIS2,THR2,CV2,RST2,OUT2,TRIG2,+5V">
-<segment>
-<wire x1="52.07" y1="-21.59" x2="52.07" y2="29.21" width="0.762" layer="92"/>
+<bus name="GND,DIS,THR_TRIG,CV,RST,OUT,VCC,DIS2,CV2,RST2,OUT2,THR2_TRIG2,+5V">
+<segment>
+<wire x1="52.07" y1="-21.59" x2="52.07" y2="39.37" width="0.762" layer="92"/>
 <wire x1="52.07" y1="-21.59" x2="86.36" y2="-21.59" width="0.762" layer="92"/>
-<wire x1="86.36" y1="-21.59" x2="86.36" y2="31.75" width="0.762" layer="92"/>
+<wire x1="86.36" y1="-21.59" x2="86.36" y2="39.37" width="0.762" layer="92"/>
+<wire x1="52.07" y1="39.37" x2="86.36" y2="39.37" width="0.762" layer="92"/>
 </segment>
 </bus>
@@
 </segment>
 <segment>
-<pinref part="IC2" gate="A" pin="GND"/>
-<wire x1="59.69" y1="-13.97" x2="52.07" y2="-13.97" width="0.1524" layer="91"/>
-</segment>
-<segment>
 <pinref part="IC1" gate="G$1" pin="GND"/>
 <wire x1="55.88" y1="13.97" x2="52.07" y2="13.97" width="0.1524" layer="91"/>
+</segment>
+<segment>
+<pinref part="555" gate="G$1" pin="/RES"/>
+<wire x1="80.01" y1="-1.27" x2="86.36" y2="-1.27" width="0.1524" layer="91"/>
+</segment>
+<segment>
+<pinref part="555" gate="G$1" pin="GND"/>
+<wire x1="80.01" y1="-13.97" x2="86.36" y2="-13.97" width="0.1524" layer="91"/>
 </segment>
 </net>
@@
 </segment>
 <segment>
-<pinref part="IC2" gate="A" pin="DIS"/>
-<wire x1="80.01" y1="-3.81" x2="86.36" y2="-3.81" width="0.1524" layer="91"/>
-</segment>
-</net>
-<net name="THR" class="0">
+<pinref part="555" gate="G$1" pin="DIS"/>
+<wire x1="59.69" y1="-6.35" x2="52.07" y2="-6.35" width="0.1524" layer="91"/>
+</segment>
+</net>
+<net name="THR_TRIG" class="0">
 <segment>
 <pinref part="IC1" gate="G$1" pin="THR"/>
@@
 </segment>
 <segment>
-<pinref part="IC2" gate="A" pin="THR"/>
-<wire x1="80.01" y1="-8.89" x2="86.36" y2="-8.89" width="0.1524" layer="91"/>
-</segment>
-<segment>
 <pinref part="R8" gate="G$1" pin="1"/>
 <pinref part="C1" gate="G$1" pin="+"/>
-<wire x1="38.1" y1="-1.27" x2="38.1" y2="-6.35" width="0.1524" layer="91"/>
-<wire x1="38.1" y1="-6.35" x2="38.1" y2="-25.4" width="0.1524" layer="91"/>
-<wire x1="52.07" y1="-6.35" x2="38.1" y2="-6.35" width="0.1524" layer="91"/>
-<junction x="38.1" y="-6.35"/>
+<wire x1="38.1" y1="-1.27" x2="38.1" y2="-10.16" width="0.1524" layer="91"/>
+<wire x1="38.1" y1="-10.16" x2="38.1" y2="-25.4" width="0.1524" layer="91"/>
+<wire x1="52.07" y1="-10.16" x2="38.1" y2="-10.16" width="0.1524" layer="91"/>
+<junction x="38.1" y="-10.16"/>
 </segment>
 <segment>
@@
 </segment>
 <segment>
-<pinref part="IC2" gate="A" pin="TR"/>
+<pinref part="555" gate="G$1" pin="TRI"/>
+<wire x1="59.69" y1="-13.97" x2="52.07" y2="-13.97" width="0.1524" layer="91"/>
+</segment>
+<segment>
+<pinref part="555" gate="G$1" pin="TRE"/>
 <wire x1="59.69" y1="1.27" x2="52.07" y2="1.27" width="0.1524" layer="91"/>
 </segment>
@@
 </segment>
 <segment>
-<pinref part="IC2" gate="A" pin="CV"/>
-<wire x1="59.69" y1="-8.89" x2="52.07" y2="-8.89" width="0.1524" layer="91"/>
-</segment>
-<segment>
 <pinref part="C3" gate="G$1" pin="1"/>
 <wire x1="55.88" y1="-21.59" x2="55.88" y2="-25.4" width="0.1524" layer="91"/>
 </segment>
-</net>
-<net name="+5V" class="0">
+<segment>
+<pinref part="555" gate="G$1" pin="CON"/>
+<wire x1="80.01" y1="-11.43" x2="86.36" y2="-11.43" width="0.1524" layer="91"/>
+</segment>
+</net>
+<net name="VCC+" class="0">
 <segment>
 <pinref part="IC1" gate="G$1" pin="RST"/>
@@
 </segment>
 <segment>
-<pinref part="IC2" gate="A" pin="R"/>
-<wire x1="59.69" y1="-3.81" x2="52.07" y2="-3.81" width="0.1524" layer="91"/>
-</segment>
-<segment>
-<wire x1="52.07" y1="27.94" x2="49.53" y2="27.94" width="0.1524" layer="91"/>
 <pinref part="SUPPLY1" gate="+5V" pin="+5V"/>
 <wire x1="19.05" y1="33.02" x2="19.05" y2="35.56" width="0.1524" layer="91"/>
@@
 <pinref part="R4" gate="G$1" pin="2"/>
 <wire x1="27.94" y1="44.45" x2="38.1" y2="44.45" width="0.1524" layer="91"/>
-<wire x1="38.1" y1="44.45" x2="49.53" y2="44.45" width="0.1524" layer="91"/>
-<wire x1="49.53" y1="44.45" x2="93.98" y2="44.45" width="0.1524" layer="91"/>
+<wire x1="38.1" y1="44.45" x2="69.85" y2="44.45" width="0.1524" layer="91"/>
+<wire x1="69.85" y1="44.45" x2="93.98" y2="44.45" width="0.1524" layer="91"/>
 <wire x1="93.98" y1="44.45" x2="102.87" y2="44.45" width="0.1524" layer="91"/>
 <wire x1="102.87" y1="44.45" x2="102.87" y2="40.64" width="0.1524" layer="91"/>
@@
 <wire x1="93.98" y1="30.48" x2="93.98" y2="44.45" width="0.1524" layer="91"/>
 <junction x="93.98" y="44.45"/>
-<wire x1="49.53" y1="27.94" x2="49.53" y2="44.45" width="0.1524" layer="91"/>
-<junction x="49.53" y="44.45"/>
+<wire x1="69.85" y1="39.37" x2="69.85" y2="44.45" width="0.1524" layer="91"/>
+<junction x="69.85" y="44.45"/>
 </segment>
 <segment>
@@
 </segment>
 <segment>
-<pinref part="IC2" gate="A" pin="V+"/>
-<wire x1="80.01" y1="-13.97" x2="86.36" y2="-13.97" width="0.1524" layer="91"/>
-</segment>
-</net>
-<net name="556IC5" class="0">
+<pinref part="555" gate="G$1" pin="VCC+"/>
+<wire x1="80.01" y1="1.27" x2="86.36" y2="1.27" width="0.1524" layer="91"/>
+</segment>
+</net>
+<net name="OUT" class="0">
 <segment>
 <pinref part="IC1" gate="G$1" pin="OUT"/>
 <wire x1="55.88" y1="19.05" x2="52.07" y2="19.05" width="0.1524" layer="91"/>
-</segment>
-<segment>
-<pinref part="IC2" gate="A" pin="Q"/>
-<wire x1="80.01" y1="1.27" x2="86.36" y2="1.27" width="0.1524" layer="91"/>
 </segment>
 <segment>
@@
 <junction x="27.94" y="11.43"/>
 </segment>
-</net>
-<net name="TRIG2" class="0">
+<segment>
+<pinref part="555" gate="G$1" pin="OUT"/>
+<wire x1="80.01" y1="-6.35" x2="86.36" y2="-6.35" width="0.1524" layer="91"/>
+</segment>
+</net>
+<net name="THR2_TRIG2" class="0">
 <segment>
 <pinref part="IC1" gate="G$1" pin="TRIG2"/>
@@
 <pinref part="R7" gate="G$1" pin="1"/>
 <pinref part="C2" gate="G$1" pin="+"/>
-<wire x1="93.98" y1="0" x2="93.98" y2="-11.43" width="0.1524" layer="91"/>
-<wire x1="93.98" y1="-11.43" x2="93.98" y2="-25.4" width="0.1524" layer="91"/>
-<wire x1="86.36" y1="-11.43" x2="93.98" y2="-11.43" width="0.1524" layer="91"/>
-<junction x="93.98" y="-11.43"/>
-</segment>
-</net>
-<net name="556IC9" class="0">
+<wire x1="93.98" y1="0" x2="93.98" y2="-19.05" width="0.1524" layer="91"/>
+<wire x1="93.98" y1="-19.05" x2="93.98" y2="-25.4" width="0.1524" layer="91"/>
+<wire x1="86.36" y1="-19.05" x2="93.98" y2="-19.05" width="0.1524" layer="91"/>
+<junction x="93.98" y="-19.05"/>
+</segment>
+</net>
+<net name="OUT2" class="0">
 <segment>
 <pinref part="IC1" gate="G$1" pin="OUT2"/>
@@
 </segment>
 </net>
-<net name="556IC11" class="0">
+<net name="CV2" class="0">
 <segment>
 <pinref part="IC1" gate="G$1" pin="CV2"/>
@@
 </segment>
 </net>
-<net name="556IC13" class="0">
+<net name="DIS2" class="0">
 <segment>
 <pinref part="IC1" gate="G$1" pin="DIS2"/>

Commit message: Revisions
Connections:
- removed net VCC+: 555.VCC+, IC1.RST, IC1.RST2, IC1.VCC, J2.PWR, R1.2, R4.2, R5.2, R6.2
- new net +5V: 555./RES, 555.VCC+, IC1.RST, IC1.RST2, IC1.VCC, J2.PWR, R1.2, R4.2, R5.2, R6.2
- net GND: no longer 555./RES
Changed lines of the file:
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@@
 <grid distance="0.05" unitdist="inch" unit="inch" style="lines" multiple="1" display="yes" altdistance="0.01" altunitdist="inch" altunit="inch"/>
 <layers>
-<layer number="1" name="Top" color="4" fill="1" visible="yes" active="no"/>
-<layer number="16" name="Bottom" color="1" fill="1" visible="yes" active="no"/>
-<layer number="17" name="Pads" color="2" fill="1" visible="yes" active="no"/>
-<layer number="18" name="Vias" color="2" fill="1" visible="yes" active="no"/>
-<layer number="19" name="Unrouted" color="6" fill="1" visible="yes" active="no"/>
-<layer number="20" name="Dimension" color="15" fill="1" visible="yes" active="no"/>
-<layer number="21" name="tPlace" color="48" fill="1" visible="yes" active="no"/>
-<layer number="22" name="bPlace" color="42" fill="1" visible="yes" active="no"/>
-<layer number="23" name="tOrigins" color="15" fill="1" visible="yes" active="no"/>
-<layer number="24" name="bOrigins" color="15" fill="1" visible="yes" active="no"/>
-<layer number="25" name="tNames" color="7" fill="1" visible="yes" active="no"/>
-<layer number="26" name="bNames" color="7" fill="1" visible="yes" active="no"/>
-<layer number="27" name="tValues" color="7" fill="1" visible="yes" active="no"/>
-<layer number="28" name="bValues" color="7" fill="1" visible="yes" active="no"/>
+<layer number="1" name="Top" color="4" fill="1" visible="no" active="no"/>
+<layer number="16" name="Bottom" color="1" fill="1" visible="no" active="no"/>
+<layer number="17" name="Pads" color="2" fill="1" visible="no" active="no"/>
+<layer number="18" name="Vias" color="2" fill="1" visible="no" active="no"/>
+<layer number="19" name="Unrouted" color="6" fill="1" visible="no" active="no"/>
+<layer number="20" name="Dimension" color="15" fill="1" visible="no" active="no"/>
+<layer number="21" name="tPlace" color="48" fill="1" visible="no" active="no"/>
+<layer number="22" name="bPlace" color="42" fill="1" visible="no" active="no"/>
+<layer number="23" name="tOrigins" color="15" fill="1" visible="no" active="no"/>
+<layer number="24" name="bOrigins" color="15" fill="1" visible="no" active="no"/>
+<layer number="25" name="tNames" color="7" fill="1" visible="no" active="no"/>
+<layer number="26" name="bNames" color="7" fill="1" visible="no" active="no"/>
+<layer number="27" name="tValues" color="7" fill="1" visible="no" active="no"/>
+<layer number="28" name="bValues" color="7" fill="1" visible="no" active="no"/>
 <layer number="29" name="tStop" color="7" fill="3" visible="no" active="no"/>
 <layer number="30" name="bStop" color="7" fill="6" visible="no" active="no"/>
@@
 <layer number="35" name="tGlue" color="7" fill="4" visible="no" active="no"/>
 <layer number="36" name="bGlue" color="7" fill="5" visible="no" active="no"/>
-<layer number="37" name="tTest" color="7" fill="1" visible="yes" active="no"/>
-<layer number="38" name="bTest" color="7" fill="1" visible="yes" active="no"/>
+<layer number="37" name="tTest" color="7" fill="1" visible="no" active="no"/>
+<layer number="38" name="bTest" color="7" fill="1" visible="no" active="no"/>
 <layer number="39" name="tKeepout" color="4" fill="11" visible="no" active="no"/>
 <layer number="40" name="bKeepout" color="1" fill="11" visible="no" active="no"/>
@@
 <layer number="44" name="Drills" color="7" fill="1" visible="no" active="no"/>
 <layer number="45" name="Holes" color="7" fill="1" visible="no" active="no"/>
-<layer number="46" name="Milling" color="3" fill="1" visible="yes" active="no"/>
-<layer number="47" name="Measures" color="7" fill="1" visible="yes" active="no"/>
-<layer number="48" name="Document" color="7" fill="1" visible="yes" active="no"/>
-<layer number="49" name="Reference" color="7" fill="1" visible="yes" active="no"/>
-<layer number="50" name="dxf" color="7" fill="1" visible="yes" active="no"/>
-<layer number="51" name="tDocu" color="7" fill="1" visible="yes" active="no"/>
-<layer number="52" name="bDocu" color="7" fill="1" visible="yes" active="no"/>
-<layer number="53" name="tGND_GNDA" color="7" fill="9" visible="yes" active="no"/>
-<layer number="54" name="bGND_GNDA" color="1" fill="9" visible="yes" active="no"/>
-<layer number="56" name="wert" color="7" fill="1" visible="yes" active="no"/>
-<layer number="57" name="tCAD" color="7" fill="1" visible="yes" active="no"/>
-<layer number="59" name="tCarbon" color="7" fill="1" visible="yes" active="no"/>
-<layer number="60" name="bCarbon" color="7" fill="1" visible="yes" active="no"/>
+<layer number="46" name="Milling" color="3" fill="1" visible="no" active="no"/>
+<layer number="47" name="Measures" color="7" fill="1" visible="no" active="no"/>
+<layer number="48" name="Document" color="7" fill="1" visible="no" active="no"/>
+<layer number="49" name="Reference" color="7" fill="1" visible="no" active="no"/>
+<layer number="50" name="dxf" color="7" fill="1" visible="no" active="no"/>
+<layer number="51" name="tDocu" color="7" fill="1" visible="no" active="no"/>
+<layer number="52" name="bDocu" color="7" fill="1" visible="no" active="no"/>
+<layer number="53" name="tGND_GNDA" color="7" fill="9" visible="no" active="no"/>
+<layer number="54" name="bGND_GNDA" color="1" fill="9" visible="no" active="no"/>
+<layer number="56" name="wert" color="7" fill="1" visible="no" active="no"/>
+<layer number="57" name="tCAD" color="7" fill="1" visible="no" active="no"/>
+<layer number="59" name="tCarbon" color="7" fill="1" visible="no" active="no"/>
+<layer number="60" name="bCarbon" color="7" fill="1" visible="no" active="no"/>
 <layer number="90" name="Modules" color="5" fill="1" visible="yes" active="yes"/>
 <layer number="91" name="Nets" color="2" fill="1" visible="yes" active="yes"/>
@@
 </class>
 </classes>
+<modules>
+<module name="YAR" prefix="" dx="30.48" dy="20.32">
+<ports>
+</ports>
+<variantdefs>
+</variantdefs>
+<parts>
+</parts>
+<sheets>
+<sheet>
+<plain>
+</plain>
+<instances>
+</instances>
+<busses>
+</busses>
+<nets>
+</nets>
+</sheet>
+</sheets>
+</module>
+</modules>
 <parts>
 <part name="IC1" library="SparkFun-AnalogIC" deviceset="556" device="KIT" value="556"/>
@@
 <bus name="GND,DIS,THR_TRIG,CV,RST,OUT,VCC,DIS2,CV2,RST2,OUT2,THR2_TRIG2,+5V">
 <segment>
-<wire x1="52.07" y1="-21.59" x2="52.07" y2="39.37" width="0.762" layer="92"/>
-<wire x1="52.07" y1="-21.59" x2="86.36" y2="-21.59" width="0.762" layer="92"/>
-<wire x1="86.36" y1="-21.59" x2="86.36" y2="39.37" width="0.762" layer="92"/>
-<wire x1="52.07" y1="39.37" x2="86.36" y2="39.37" width="0.762" layer="92"/>
+<wire x1="52.07" y1="-21.59" x2="52.07" y2="39.37" width="0.381" layer="92"/>
+<wire x1="52.07" y1="-21.59" x2="86.36" y2="-21.59" width="0.381" layer="92"/>
+<wire x1="86.36" y1="-21.59" x2="86.36" y2="39.37" width="0.381" layer="92"/>
+<wire x1="52.07" y1="39.37" x2="86.36" y2="39.37" width="0.381" layer="92"/>
 </segment>
 </bus>
@@
 <wire x1="69.85" y1="-21.59" x2="69.85" y2="-35.56" width="0.1524" layer="91"/>
 <junction x="69.85" y="-35.56"/>
+<label x="71.12" y="-26.67" size="1.778" layer="95"/>
 </segment>
 <segment>
 <pinref part="IC1" gate="G$1" pin="GND"/>
 <wire x1="55.88" y1="13.97" x2="52.07" y2="13.97" width="0.1524" layer="91"/>
-</segment>
-<segment>
-<pinref part="555" gate="G$1" pin="/RES"/>
-<wire x1="80.01" y1="-1.27" x2="86.36" y2="-1.27" width="0.1524" layer="91"/>
 </segment>
 <segment>
@@
 </segment>
 </net>
-<net name="VCC+" class="0">
+<net name="+5V" class="0">
 <segment>
 <pinref part="IC1" gate="G$1" pin="RST"/>
@@
 <wire x1="80.01" y1="1.27" x2="86.36" y2="1.27" width="0.1524" layer="91"/>
 </segment>
+<segment>
+<pinref part="555" gate="G$1" pin="/RES"/>
+<wire x1="80.01" y1="-1.27" x2="86.36" y2="-1.27" width="0.1524" layer="91"/>
+</segment>
 </net>
 <net name="OUT" class="0">
@@
 </sheet>
 </sheets>
+<errors>
+</errors>
 </schematic>
 </drawing>
